Commit message: Having some issues with the sensors.

File: data/va_kuka/arm/va_iiwa_model.urdf (robot description, URDF)
Before this commit: robot lbr_iiwa, 8 links, 7 joints
Links:
- added link iiwa7_link_ft300_mounting_plate; collision mesh filename=package://robotiq_ft_sensor/meshes/collision/mountings/robo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; visual mesh filename=package://robotiq_ft_sensor/meshes/visual/mountings/robotiq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
- added link iiwa7_link_ft300_sensor, mass 0.300; collision mesh filename=package://robotiq_ft_sensor/meshes/collision/robotiq_ft300.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; visual mesh filename=package://robotiq_ft_sensor/meshes/visual/robotiq_ft300.STL
- added link iiwa7_robotiq_ft_frame_id
Joints:
- added joint iiwa7_joint_ft300_mounting_plate: type fixed, parent iiwa7_link_ft300_mounting_plate, child iiwa7_link_ft300_sensor, origin xyz=0 0 0.0415 rpy=0 ${pi} 0
- added joint iiwa7_joint_ft_mount: type fixed, parent lbr_iiwa_link_7, child iiwa7_link_ft300_mounting_plate, origin xyz=0 0 0.0415 rpy=0 0 0
- added joint iiwa7_measurement_joint: type fixed, parent iiwa7_ft300_sensor, child iiwa7_robotiq_ft_frame_id, origin xyz=0 0 0 rpy=0 ${pi} ${-pi/2}

File: data/va_kuka/va_iiwa_model.urdf (robot description, URDF)
Before this commit: robot lbr_iiwa, 8 links, 7 joints
Links:
- added link iiwa7_link_ft300_mounting_plate, mass 0.3; collision mesh filename=robotiq_ft_sensor/meshes/collision/mountings/robotiq_ft300-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; visual mesh filename=robotiq_ft_sensor/meshes/visual/mountings/robotiq_ft300-G-0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
- added link iiwa7_link_ft300_sensor, mass 0.300; collision mesh filename=robotiq_ft_sensor/meshes/collision/robotiq_ft300.STL; visual mesh filename=robotiq_ft_sensor/meshes/visual/robotiq_ft300.STL
- added link iiwa7_robotiq_ft_frame_id
Joints:
- added joint iiwa7_joint_ft300_mounting_plate: type fixed, parent iiwa7_link_ft300_mounting_plate, child iiwa7_link_ft300_sensor, origin xyz=0 0 0.0415 rpy=0 ${pi} 0
- added joint iiwa7_joint_ft_mount: type fixed, parent lbr_iiwa_link_7, child iiwa7_link_ft300_mounting_plate, origin xyz=0 0 0.0415 rpy=0 0 0
- added joint iiwa7_measurement_joint: type fixed, parent iiwa7_ft300_sensor, child iiwa7_robotiq_ft_frame_id, origin xyz=0 0 0 rpy=0 ${pi} ${-pi/2}
