Commit message: Discovered code was exiting from va_sim.py.

File: data/va_kuka/va_iiwa_model.urdf (robot description, URDF)
Before this commit: robot lbr_iiwa, 11 links, 10 joints
Links:
- removed link iiwa7_robotiq_ft_frame_id
- link iiwa7_link_ft300_mounting_plate: mass 0.3 -> 0.03
Joints:
- removed joint iiwa7_measurement_joint

Commit message: Successfully simulated force_sensor.

File: data/va_kuka/va_iiwa_model.urdf (robot description, URDF)
Before this commit: robot lbr_iiwa, 10 links, 9 joints
Joints:
- removed joint iiwa7_joint_ft_mount
- added joint iiwa7_joint_ft300_sensor: type fixed, parent iiwa7_link_ft300_mounting_plate, child iiwa7_link_ft300_sensor, origin xyz=0 0 0 rpy=0 ${pi} 0
- joint iiwa7_joint_ft300_mounting_plate: child iiwa7_link_ft300_sensor -> iiwa7_link_ft300_mounting_plate; origin xyz=0 0 0.0415 rpy=0 ${pi} 0 -> xyz=0 0 0.0415 rpy=0 0 0; parent iiwa7_link_ft300_mounting_plate -> lbr_iiwa_link_7
