Commit message: Simulated gripper, but gripper still in weird shape.

File: data/va_kuka/robotiq_85_gripper/robotiq_85_gripper.urdf.xacro (robot description, xacro)
@@ -3,11 +3,11 @@
     <xacro:include filename="$(find robotiq_85_description)/urdf/robotiq_85_gripper.transmission.xacro" />
     <xacro:macro name="robotiq_85_gripper" params="prefix parent robotNS *origin">
-        <joint name="iiwa7_gripper_base_joint" type="fixed">
+        <joint name="${prefix}gripper_base_joint" type="fixed">
             <xacro:insert_block name="origin"/>
             <parent link="${parent}"/>
-            <child link="iiwa7_gripper_base_link"/>
+            <child link="${prefix}gripper_base_link"/>
             <xacro:insert_block name="origin"/>
         </joint>
-        <link name="iiwa7_gripper_base_link">
+        <link name="${prefix}gripper_base_link">
             <visual>
                 <geometry>
@@ -28,28 +28,28 @@
             </inertial>
         </link>
-        <gazebo reference="iiwa7_gripper_base_link">
-            <implicitSpringDamper>1</implicitSpringDamper>
-            <mu1>100000</mu1>
-            <mu2>100000</mu2>
-            <kp>100000000.0</kp>
-            <kd>1.0</kd>
-        </gazebo>
-        <joint name="iiwa7_gripper_finger1_joint" type="revolute">
-            <parent link="iiwa7_gripper_base_link"/>
-            <child link="iiwa7_gripper_finger1_knuckle_link"/>
+        <gazebo reference="${prefix}gripper_base_link">
+            <implicitSpringDamper>1</implicitSpringDamper>
+            <mu1>100000</mu1>
+            <mu2>100000</mu2>
+            <kp>100000000.0</kp>
+            <kd>1.0</kd>
+        </gazebo>
+        <joint name="${prefix}gripper_finger1_joint" type="revolute">
+            <parent link="${prefix}gripper_base_link"/>
+            <child link="${prefix}gripper_finger1_knuckle_link"/>
             <axis xyz="0 0 1"/>
             <origin rpy="${pi} 0.0 0.0" xyz="0.05490451627 0.03060114443 0.0"/>
             <limit lower="0.0" upper="0.804" velocity="2.0" effort="1000"/>
-            <mimic joint="iiwa7_gripper_finger1_inner_knuckle_joint" offset="0"/>
-        </joint>
-        <joint name="iiwa7_gripper_finger2_joint" type="revolute">
-            <parent link="iiwa7_gripper_base_link"/>
-            <child link="iiwa7_gripper_finger2_knuckle_link"/>
+            <mimic joint="${prefix}gripper_finger1_inner_knuckle_joint" offset="0"/>
+        </joint>
+        <joint name="${prefix}gripper_finger2_joint" type="revolute">
+            <parent link="${prefix}gripper_base_link"/>
+            <child link="${prefix}gripper_finger2_knuckle_link"/>
             <axis xyz="0 0 1"/>
             <origin rpy="0.0 0.0 0.0" xyz="0.05490451627 -0.03060114443 0.0"/>
             <limit lower="0.0" upper="1.0" velocity="100.0" effort="1000"/>
-            <mimic joint="iiwa7_gripper_finger1_inner_knuckle_joint" offset="0" multiplier="1"/>
-        </joint>
-        <link name="iiwa7_gripper_finger1_knuckle_link">
+            <mimic joint="${prefix}gripper_finger1_inner_knuckle_joint" offset="0" multiplier="1"/>
+        </joint>
+        <link name="${prefix}gripper_finger1_knuckle_link">
             <visual>
                 <geometry>
@@ -70,13 +70,13 @@
             </inertial>
         </link>
-        <gazebo reference="iiwa7_gripper_finger1_knuckle_link">
-            <implicitSpringDamper>1</implicitSpringDamper>
-            <mu1>100000</mu1>
-            <mu2>100000</mu2>
-            <kp>100000000.0</kp>
-            <kd>1.0</kd>
-            <self_collide>0</self_collide>
-        </gazebo>
-        <link name="iiwa7_gripper_finger2_knuckle_link">
+        <gazebo reference="${prefix}gripper_finger1_knuckle_link">
+            <implicitSpringDamper>1</implicitSpringDamper>
+            <mu1>100000</mu1>
+            <mu2>100000</mu2>
+            <kp>100000000.0</kp>
+            <kd>1.0</kd>
+            <self_collide>0</self_collide>
+        </gazebo>
+        <link name="${prefix}gripper_finger2_knuckle_link">
             <visual>
                 <geometry>
@@ -97,23 +97,23 @@
             </inertial>
         </link>
-        <gazebo reference="iiwa7_gripper_finger2_knuckle_link">
-            <implicitSpringDamper>1</implicitSpringDamper>
-            <mu1>100000</mu1>
-            <mu2>100000</mu2>
-            <kp>100000000.0</kp>
-            <kd>1.0</kd>
-            <self_collide>0</self_collide>
-        </gazebo>
-        <joint name="iiwa7_gripper_finger1_finger_joint" type="fixed">
-            <parent link="iiwa7_gripper_finger1_knuckle_link"/>
-            <child link="iiwa7_gripper_finger1_finger_link"/>
+        <gazebo reference="${prefix}gripper_finger2_knuckle_link">
+            <implicitSpringDamper>1</implicitSpringDamper>
+            <mu1>100000</mu1>
+            <mu2>100000</mu2>
+            <kp>100000000.0</kp>
+            <kd>1.0</kd>
+            <self_collide>0</self_collide>
+        </gazebo>
+        <joint name="${prefix}gripper_finger1_finger_joint" type="fixed">
+            <parent link="${prefix}gripper_finger1_knuckle_link"/>
+            <child link="${prefix}gripper_finger1_finger_link"/>
             <origin xyz="-0.00408552455 -0.03148604435 0.0" rpy="0 0 0" />
         </joint>
-        <joint name="iiwa7_gripper_finger2_finger_joint" type="fixed">
-            <parent link="iiwa7_gripper_finger2_knuckle_link"/>
-            <child link="iiwa7_gripper_finger2_finger_link"/>
+        <joint name="${prefix}gripper_finger2_finger_joint" type="fixed">
+            <parent link="${prefix}gripper_finger2_knuckle_link"/>
+            <child link="${prefix}gripper_finger2_finger_link"/>
             <origin xyz="-0.00408552455 -0.03148604435 0.0" rpy="0 0 0" />
         </joint>
-        <link name="iiwa7_gripper_finger1_finger_link">
+        <link name="${prefix}gripper_finger1_finger_link">
             <visual>
                 <geometry>
@@ -134,13 +134,13 @@
             </inertial>
         </link>
-        <gazebo reference="iiwa7_gripper_finger1_finger_link">
-            <implicitSpringDamper>1</implicitSpringDamper>
-            <mu1>100000</mu1>
-            <mu2>100000</mu2>
-            <kp>100000000.0</kp>
-            <kd>1.0</kd>
-            <self_collide>0</self_collide>
-        </gazebo>
-        <link name="iiwa7_gripper_finger2_finger_link">
+        <gazebo reference="${prefix}gripper_finger1_finger_link">
+            <implicitSpringDamper>1</implicitSpringDamper>
+            <mu1>100000</mu1>
+            <mu2>100000</mu2>
+            <kp>100000000.0</kp>
+            <kd>1.0</kd>
+            <self_collide>0</self_collide>
+        </gazebo>
+        <link name="${prefix}gripper_finger2_finger_link">
             <visual>
                 <geometry>
@@ -161,28 +161,28 @@
             </inertial>
         </link>
-        <gazebo reference="iiwa7_gripper_finger2_finger_link">
-            <implicitSpringDamper>1</implicitSpringDamper>
-            <mu1>100000</mu1>
-            <mu2>100000</mu2>
-            <kp>100000000.0</kp>
-            <kd>1.0</kd>
-            <self_collide>0</self_collide>
-        </gazebo>
-        <joint name="iiwa7_gripper_finger1_inner_knuckle_joint" type="revolute">
-            <parent link="iiwa7_gripper_base_link"/>
-            <child link="iiwa7_gripper_finger1_inner_knuckle_link"/>
+        <gazebo reference="${prefix}gripper_finger2_finger_link">
+            <implicitSpringDamper>1</implicitSpringDamper>
+            <mu1>100000</mu1>
+            <mu2>100000</mu2>
+            <kp>100000000.0</kp>
+            <kd>1.0</kd>
+            <self_collide>0</self_collide>
+        </gazebo>
+        <joint name="${prefix}gripper_finger1_inner_knuckle_joint" type="revolute">
+            <parent link="${prefix}gripper_base_link"/>
+            <child link="${prefix}gripper_finger1_inner_knuckle_link"/>
             <axis xyz="0 0 1"/>
             <origin xyz="0.06142 0.0127 0" rpy="${pi} 0.0 0.0" />
             <limit lower="0.0" upper="1.0" velocity="100.0" effort="0.1"/>
         </joint>
-        <joint name="iiwa7_gripper_finger2_inner_knuckle_joint" type="revolute">
-            <parent link="iiwa7_gripper_base_link"/>
-            <child link="iiwa7_gripper_finger2_inner_knuckle_link"/>
+        <joint name="${prefix}gripper_finger2_inner_knuckle_joint" type="revolute">
+            <parent link="${prefix}gripper_base_link"/>
+            <child link="${prefix}gripper_finger2_inner_knuckle_link"/>
             <axis xyz="0 0 1"/>
             <origin xyz="0.06142 -0.0127 0" rpy="0 0 0"/>
             <limit lower="0.0" upper="1.0" velocity="100.0" effort="0.1"/>
-            <mimic joint="iiwa7_gripper_finger1_inner_knuckle_joint" offset="0"/>
-        </joint>
-        <link name="iiwa7_gripper_finger1_inner_knuckle_link">
+            <mimic joint="${prefix}gripper_finger1_inner_knuckle_joint" offset="0"/>
+        </joint>
+        <link name="${prefix}gripper_finger1_inner_knuckle_link">
             <visual>
                 <geometry>
@@ -203,13 +203,13 @@
             </inertial>
         </link>
-        <gazebo reference="iiwa7_gripper_finger1_inner_knuckle_link">
-            <implicitSpringDamper>1</implicitSpringDamper>
-            <mu1>100000</mu1>
-            <mu2>100000</mu2>
-            <kp>100000000.0</kp>
-            <kd>1.0</kd>
-            <self_collide>0</self_collide>
-        </gazebo>
-        <link name="iiwa7_gripper_finger2_inner_knuckle_link">
+        <gazebo reference="${prefix}gripper_finger1_inner_knuckle_link">
+            <implicitSpringDamper>1</implicitSpringDamper>
+            <mu1>100000</mu1>
+            <mu2>100000</mu2>
+            <kp>100000000.0</kp>
+            <kd>1.0</kd>
+            <self_collide>0</self_collide>
+        </gazebo>
+        <link name="${prefix}gripper_finger2_inner_knuckle_link">
             <visual>
                 <geometry>
@@ -230,29 +230,29 @@
             </inertial>
         </link>
-        <gazebo reference="iiwa7_gripper_finger2_inner_knuckle_link">
-            <implicitSpringDamper>1</implicitSpringDamper>
-            <mu1>100000</mu1>
-            <mu2>100000</mu2>
-            <kp>100000000.0</kp>
-            <kd>1.0</kd>
-            <self_collide>0</self_collide>
-        </gazebo>
-        <joint name="iiwa7_gripper_finger1_finger_tip_joint" type="revolute">
-            <parent link="iiwa7_gripper_finger1_inner_knuckle_link"/>
-            <child link="iiwa7_gripper_finger1_finger_tip_link"/>
+        <gazebo reference="${prefix}gripper_finger2_inner_knuckle_link">
+            <implicitSpringDamper>1</implicitSpringDamper>
+            <mu1>100000</mu1>
+            <mu2>100000</mu2>
+            <kp>100000000.0</kp>
+            <kd>1.0</kd>
+            <self_collide>0</self_collide>
+        </gazebo>
+        <joint name="${prefix}gripper_finger1_finger_tip_joint" type="revolute">
+            <parent link="${prefix}gripper_finger1_inner_knuckle_link"/>
+            <child link="${prefix}gripper_finger1_finger_tip_link"/>
             <axis xyz="0 0 1"/>
             <origin xyz="0.04303959807 -0.03759940821 0.0" rpy="0.0 0.0 0.0"/>
             <limit lower="-1.0" upper="0.0" velocity="100.0" effort="0.1"/>
-            <mimic joint="iiwa7_gripper_finger1_inner_knuckle_joint" multiplier="-1" offset="0"/>
-        </joint>
-        <joint name="iiwa7_gripper_finger2_finger_tip_joint" type="revolute">
-            <parent link="iiwa7_gripper_finger2_inner_knuckle_link"/>
-            <child link="iiwa7_gripper_finger2_finger_tip_link"/>
+            <mimic joint="${prefix}gripper_finger1_inner_knuckle_joint" multiplier="-1" offset="0"/>
+        </joint>
+        <joint name="${prefix}gripper_finger2_finger_tip_joint" type="revolute">
+            <parent link="${prefix}gripper_finger2_inner_knuckle_link"/>
+            <child link="${prefix}gripper_finger2_finger_tip_link"/>
             <axis xyz="0 0 1"/>
             <origin rpy="0.0 0.0 0.0" xyz="0.04303959807 -0.03759940821  0.0"/>
             <limit lower="-1.0" upper="0.0" velocity="100.0" effort="0.1"/>
-            <mimic joint="iiwa7_gripper_finger1_inner_knuckle_joint" multiplier="-1" offset="0"/>
-        </joint>
-        <link name="iiwa7_gripper_finger1_finger_tip_link">
+            <mimic joint="${prefix}gripper_finger1_inner_knuckle_joint" multiplier="-1" offset="0"/>
+        </joint>
+        <link name="${prefix}gripper_finger1_finger_tip_link">
             <visual>
                 <geometry>
@@ -273,13 +273,13 @@
             </inertial>
         </link>
-        <gazebo reference="iiwa7_gripper_finger1_finger_tip_link">
-            <implicitSpringDamper>1</implicitSpringDamper>
-            <mu1>100000</mu1>
-            <mu2>100000</mu2>
-            <kp>100000000.0</kp>
-            <kd>1.0</kd>
-            <self_collide>0</self_collide>
-        </gazebo>
-        <link name="iiwa7_gripper_finger2_finger_tip_link">
+        <gazebo reference="${prefix}gripper_finger1_finger_tip_link">
+            <implicitSpringDamper>1</implicitSpringDamper>
+            <mu1>100000</mu1>
+            <mu2>100000</mu2>
+            <kp>100000000.0</kp>
+            <kd>1.0</kd>
+            <self_collide>0</self_collide>
+        </gazebo>
+        <link name="${prefix}gripper_finger2_finger_tip_link">
             <visual>
                 <geometry>
@@ -300,13 +300,13 @@
             </inertial>
         </link>
-        <gazebo reference="iiwa7_gripper_finger2_finger_tip_link">
-            <implicitSpringDamper>1</implicitSpringDamper>
-            <mu1>100000</mu1>
-            <mu2>100000</mu2>
-            <kp>100000000.0</kp>
-            <kd>1.0</kd>
-            <self_collide>0</self_collide>
-        </gazebo>
-        <xacro:robotiq_85_gripper_transmission prefix="iiwa7_" />
+        <gazebo reference="${prefix}gripper_finger2_finger_tip_link">
+            <implicitSpringDamper>1</implicitSpringDamper>
+            <mu1>100000</mu1>
+            <mu2>100000</mu2>
+            <kp>100000000.0</kp>
+            <kd>1.0</kd>
+            <self_collide>0</self_collide>
+        </gazebo>
+        <xacro:robotiq_85_gripper_transmission prefix="${prefix}" />
         <gazebo>
             <plugin name="gazebo_grasp_fix" filename="libgazebo_grasp_fix.so">

File: data/va_kuka/va_iiwa_model.urdf (robot description, URDF)
Before this commit: robot lbr_iiwa, 10 links, 9 joints
Links:
- added link iiwa7_gripper_base_link, mass 0.636951; collision mesh filename=robotiq_85_gripper/meshes/collision/robotiq_85_base_link.stl; visual mesh filename=robotiq_85_gripper/meshes/visual/robotiq_85_base_link.dae
- added link iiwa7_gripper_finger1_finger_link, mass 0.027309; collision mesh filename=robotiq_85_gripper/meshes/collision/robotiq_85_finger_link.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; visual mesh filename=robotiq_85_gripper/meshes/visual/robotiq_85_finger_link.dae
- added link iiwa7_gripper_finger1_finger_tip_link, mass 0.019555; collision mesh filename=robotiq_85_gripper/meshes/collision/robotiq_85_finger_tip_l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; visual mesh filename=robotiq_85_gripper/meshes/visual/robotiq_85_finger_tip_link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
- added link iiwa7_gripper_finger1_inner_knuckle_link, mass 0.029951; collision mesh filename=robotiq_85_gripper/meshes/collision/robotiq_85_inner_knuckl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; visual mesh filename=robotiq_85_gripper/meshes/visual/robotiq_85_inner_knuckle_l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
- added link iiwa7_gripper_finger1_knuckle_link, mass 0.018491; collision mesh filename=robotiq_85_gripper/meshes/collision/robotiq_85_knuckle_link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; visual mesh filename=robotiq_85_gripper/meshes/visual/robotiq_85_knuckle_link.dae
- added link iiwa7_gripper_finger2_finger_link, mass 0.027309; collision mesh filename=robotiq_85_gripper/meshes/collision/robotiq_85_finger_link.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; visual mesh filename=robotiq_85_gripper/meshes/visual/robotiq_85_finger_link.dae
- added link iiwa7_gripper_finger2_finger_tip_link, mass 0.019555; collision mesh filename=robotiq_85_gripper/meshes/collision/robotiq_85_finger_tip_l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; visual mesh filename=robotiq_85_gripper/meshes/visual/robotiq_85_finger_tip_link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
- added link iiwa7_gripper_finger2_inner_knuckle_link, mass 0.029951; collision mesh filename=robotiq_85_gripper/meshes/collision/robotiq_85_inner_knuckl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; visual mesh filename=robotiq_85_gripper/meshes/visual/robotiq_85_inner_knuckle_l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
- added link iiwa7_gripper_finger2_knuckle_link, mass 0.018491; collision mesh filename=robotiq_85_gripper/meshes/collision/robotiq_85_knuckle_link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; visual mesh filename=robotiq_85_gripper/meshes/visual/robotiq_85_knuckle_link.dae
- link iiwa7_link_ft300_mounting_plate: geometry collision mesh filename=robotiq_ft300_sensor/meshes/collision/mountings/robotiq_ft3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; visual mesh filename=robotiq_ft300_sensor/meshes/visual/mountings/robotiq_ft300-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
- link iiwa7_link_ft300_sensor: geometry collision mesh filename=robotiq_ft300_sensor/meshes/collision/robotiq_ft300.STL; visual mesh filename=robotiq_ft300_sensor/meshes/visual/robotiq_ft300.STL
Joints:
- added joint iiwa7_gripper_base_joint: type fixed, parent iiwa7_link_ft300_sensor, child iiwa7_gripper_base_link, origin xyz=0 0 0 rpy=0 -1.571 0
- added joint iiwa7_gripper_finger1_finger_joint: type fixed, parent iiwa7_gripper_finger1_knuckle_link, child iiwa7_gripper_finger1_finger_link, origin xyz=-0.00408552455 -0.03148604435 0.0 rpy=0 0 0
- added joint iiwa7_gripper_finger1_finger_tip_joint: type revolute, parent iiwa7_gripper_finger1_inner_knuckle_link, child iiwa7_gripper_finger1_finger_tip_link, origin xyz=0.04303959807 -0.03759940821 0.0 rpy=0.0 0.0 0.0, axis 0 0 1, limit lower=-1.0 upper=0.0 effort=0.1 velocity=100.0, mimic joint=iiwa7_gripper_finger1_inner_knuckle_joint multiplier=-1 offset=0
- added joint iiwa7_gripper_finger1_inner_knuckle_joint: type revolute, parent iiwa7_gripper_base_link, child iiwa7_gripper_finger1_inner_knuckle_link, origin xyz=0.06142 0.0127 0 rpy=${pi} 0.0 0.0, axis 0 0 1, limit lower=0.0 upper=1.0 effort=0.1 velocity=100.0
- added joint iiwa7_gripper_finger1_joint: type revolute, parent iiwa7_gripper_base_link, child iiwa7_gripper_finger1_knuckle_link, origin xyz=0.05490451627 0.03060114443 0.0 rpy=${pi} 0.0 0.0, axis 0 0 1, limit lower=0.0 upper=0.804 effort=1000 velocity=2.0, mimic joint=iiwa7_gripper_finger1_inner_knuckle_joint offset=0
- added joint iiwa7_gripper_finger2_finger_joint: type fixed, parent iiwa7_gripper_finger2_knuckle_link, child iiwa7_gripper_finger2_finger_link, origin xyz=-0.00408552455 -0.03148604435 0.0 rpy=0 0 0
- added joint iiwa7_gripper_finger2_finger_tip_joint: type revolute, parent iiwa7_gripper_finger2_inner_knuckle_link, child iiwa7_gripper_finger2_finger_tip_link, origin xyz=0.04303959807 -0.03759940821  0.0 rpy=0.0 0.0 0.0, axis 0 0 1, limit lower=-1.0 upper=0.0 effort=0.1 velocity=100.0, mimic joint=iiwa7_gripper_finger1_inner_knuckle_joint multiplier=-1 offset=0
- added joint iiwa7_gripper_finger2_inner_knuckle_joint: type revolute, parent iiwa7_gripper_base_link, child iiwa7_gripper_finger2_inner_knuckle_link, origin xyz=0.06142 -0.0127 0 rpy=0 0 0, axis 0 0 1, limit lower=0.0 upper=1.0 effort=0.1 velocity=100.0, mimic joint=iiwa7_gripper_finger1_inner_knuckle_joint offset=0
- added joint iiwa7_gripper_finger2_joint: type revolute, parent iiwa7_gripper_base_link, child iiwa7_gripper_finger2_knuckle_link, origin xyz=0.05490451627 -0.03060114443 0.0 rpy=0.0 0.0 0.0, axis 0 0 1, limit lower=0.0 upper=1.0 effort=1000 velocity=100.0, mimic joint=iiwa7_gripper_finger1_inner_knuckle_joint multiplier=1 offset=0
