Commit message: Cleaned up files.

File: data/va_kuka/robotiq_85_gripper/robotiq_85_gripper.urdf.xacro (robot description, xacro)
@@ -3,11 +3,11 @@
     <xacro:include filename="$(find robotiq_85_description)/urdf/robotiq_85_gripper.transmission.xacro" />
     <xacro:macro name="robotiq_85_gripper" params="prefix parent robotNS *origin">
-        <joint name="${prefix}gripper_base_joint" type="fixed">
+        <joint name="iiwa7_gripper_base_joint" type="fixed">
             <xacro:insert_block name="origin"/>
             <parent link="${parent}"/>
-            <child link="${prefix}gripper_base_link"/>
+            <child link="iiwa7_gripper_base_link"/>
             <xacro:insert_block name="origin"/>
         </joint>
-        <link name="${prefix}gripper_base_link">
+        <link name="iiwa7_gripper_base_link">
             <visual>
                 <geometry>
@@ -28,28 +28,28 @@
             </inertial>
         </link>
-        <gazebo reference="${prefix}gripper_base_link">
-            <implicitSpringDamper>1</implicitSpringDamper>
-            <mu1>100000</mu1>
-            <mu2>100000</mu2>
-            <kp>100000000.0</kp>
-            <kd>1.0</kd>
-        </gazebo>
-        <joint name="${prefix}gripper_finger1_joint" type="revolute">
-            <parent link="${prefix}gripper_base_link"/>
-            <child link="${prefix}gripper_finger1_knuckle_link"/>
+        <gazebo reference="iiwa7_gripper_base_link">
+            <implicitSpringDamper>1</implicitSpringDamper>
+            <mu1>100000</mu1>
+            <mu2>100000</mu2>
+            <kp>100000000.0</kp>
+            <kd>1.0</kd>
+        </gazebo>
+        <joint name="iiwa7_gripper_finger1_joint" type="revolute">
+            <parent link="iiwa7_gripper_base_link"/>
+            <child link="iiwa7_gripper_finger1_knuckle_link"/>
             <axis xyz="0 0 1"/>
             <origin rpy="${pi} 0.0 0.0" xyz="0.05490451627 0.03060114443 0.0"/>
             <limit lower="0.0" upper="0.804" velocity="2.0" effort="1000"/>
-            <mimic joint="${prefix}gripper_finger1_inner_knuckle_joint" offset="0"/>
-        </joint>
-        <joint name="${prefix}gripper_finger2_joint" type="revolute">
-            <parent link="${prefix}gripper_base_link"/>
-            <child link="${prefix}gripper_finger2_knuckle_link"/>
+            <mimic joint="iiwa7_gripper_finger1_inner_knuckle_joint" offset="0"/>
+        </joint>
+        <joint name="iiwa7_gripper_finger2_joint" type="revolute">
+            <parent link="iiwa7_gripper_base_link"/>
+            <child link="iiwa7_gripper_finger2_knuckle_link"/>
             <axis xyz="0 0 1"/>
             <origin rpy="0.0 0.0 0.0" xyz="0.05490451627 -0.03060114443 0.0"/>
             <limit lower="0.0" upper="1.0" velocity="100.0" effort="1000"/>
-            <mimic joint="${prefix}gripper_finger1_inner_knuckle_joint" offset="0" multiplier="1"/>
-        </joint>
-        <link name="${prefix}gripper_finger1_knuckle_link">
+            <mimic joint="iiwa7_gripper_finger1_inner_knuckle_joint" offset="0" multiplier="1"/>
+        </joint>
+        <link name="iiwa7_gripper_finger1_knuckle_link">
             <visual>
                 <geometry>
@@ -70,13 +70,13 @@
             </inertial>
         </link>
-        <gazebo reference="${prefix}gripper_finger1_knuckle_link">
-            <implicitSpringDamper>1</implicitSpringDamper>
-            <mu1>100000</mu1>
-            <mu2>100000</mu2>
-            <kp>100000000.0</kp>
-            <kd>1.0</kd>
-            <self_collide>0</self_collide>
-        </gazebo>
-        <link name="${prefix}gripper_finger2_knuckle_link">
+        <gazebo reference="iiwa7_gripper_finger1_knuckle_link">
+            <implicitSpringDamper>1</implicitSpringDamper>
+            <mu1>100000</mu1>
+            <mu2>100000</mu2>
+            <kp>100000000.0</kp>
+            <kd>1.0</kd>
+            <self_collide>0</self_collide>
+        </gazebo>
+        <link name="iiwa7_gripper_finger2_knuckle_link">
             <visual>
                 <geometry>
@@ -97,23 +97,23 @@
             </inertial>
         </link>
-        <gazebo reference="${prefix}gripper_finger2_knuckle_link">
-            <implicitSpringDamper>1</implicitSpringDamper>
-            <mu1>100000</mu1>
-            <mu2>100000</mu2>
-            <kp>100000000.0</kp>
-            <kd>1.0</kd>
-            <self_collide>0</self_collide>
-        </gazebo>
-        <joint name="${prefix}gripper_finger1_finger_joint" type="fixed">
-            <parent link="${prefix}gripper_finger1_knuckle_link"/>
-            <child link="${prefix}gripper_finger1_finger_link"/>
+        <gazebo reference="iiwa7_gripper_finger2_knuckle_link">
+            <implicitSpringDamper>1</implicitSpringDamper>
+            <mu1>100000</mu1>
+            <mu2>100000</mu2>
+            <kp>100000000.0</kp>
+            <kd>1.0</kd>
+            <self_collide>0</self_collide>
+        </gazebo>
+        <joint name="iiwa7_gripper_finger1_finger_joint" type="fixed">
+            <parent link="iiwa7_gripper_finger1_knuckle_link"/>
+            <child link="iiwa7_gripper_finger1_finger_link"/>
             <origin xyz="-0.00408552455 -0.03148604435 0.0" rpy="0 0 0" />
         </joint>
-        <joint name="${prefix}gripper_finger2_finger_joint" type="fixed">
-            <parent link="${prefix}gripper_finger2_knuckle_link"/>
-            <child link="${prefix}gripper_finger2_finger_link"/>
+        <joint name="iiwa7_gripper_finger2_finger_joint" type="fixed">
+            <parent link="iiwa7_gripper_finger2_knuckle_link"/>
+            <child link="iiwa7_gripper_finger2_finger_link"/>
             <origin xyz="-0.00408552455 -0.03148604435 0.0" rpy="0 0 0" />
         </joint>
-        <link name="${prefix}gripper_finger1_finger_link">
+        <link name="iiwa7_gripper_finger1_finger_link">
             <visual>
                 <geometry>
@@ -134,13 +134,13 @@
             </inertial>
         </link>
-        <gazebo reference="${prefix}gripper_finger1_finger_link">
-            <implicitSpringDamper>1</implicitSpringDamper>
-            <mu1>100000</mu1>
-            <mu2>100000</mu2>
-            <kp>100000000.0</kp>
-            <kd>1.0</kd>
-            <self_collide>0</self_collide>
-        </gazebo>
-        <link name="${prefix}gripper_finger2_finger_link">
+        <gazebo reference="iiwa7_gripper_finger1_finger_link">
+            <implicitSpringDamper>1</implicitSpringDamper>
+            <mu1>100000</mu1>
+            <mu2>100000</mu2>
+            <kp>100000000.0</kp>
+            <kd>1.0</kd>
+            <self_collide>0</self_collide>
+        </gazebo>
+        <link name="iiwa7_gripper_finger2_finger_link">
             <visual>
                 <geometry>
@@ -161,28 +161,28 @@
             </inertial>
         </link>
-        <gazebo reference="${prefix}gripper_finger2_finger_link">
-            <implicitSpringDamper>1</implicitSpringDamper>
-            <mu1>100000</mu1>
-            <mu2>100000</mu2>
-            <kp>100000000.0</kp>
-            <kd>1.0</kd>
-            <self_collide>0</self_collide>
-        </gazebo>
-        <joint name="${prefix}gripper_finger1_inner_knuckle_joint" type="revolute">
-            <parent link="${prefix}gripper_base_link"/>
-            <child link="${prefix}gripper_finger1_inner_knuckle_link"/>
+        <gazebo reference="iiwa7_gripper_finger2_finger_link">
+            <implicitSpringDamper>1</implicitSpringDamper>
+            <mu1>100000</mu1>
+            <mu2>100000</mu2>
+            <kp>100000000.0</kp>
+            <kd>1.0</kd>
+            <self_collide>0</self_collide>
+        </gazebo>
+        <joint name="iiwa7_gripper_finger1_inner_knuckle_joint" type="revolute">
+            <parent link="iiwa7_gripper_base_link"/>
+            <child link="iiwa7_gripper_finger1_inner_knuckle_link"/>
             <axis xyz="0 0 1"/>
             <origin xyz="0.06142 0.0127 0" rpy="${pi} 0.0 0.0" />
             <limit lower="0.0" upper="1.0" velocity="100.0" effort="0.1"/>
         </joint>
-        <joint name="${prefix}gripper_finger2_inner_knuckle_joint" type="revolute">
-            <parent link="${prefix}gripper_base_link"/>
-            <child link="${prefix}gripper_finger2_inner_knuckle_link"/>
+        <joint name="iiwa7_gripper_finger2_inner_knuckle_joint" type="revolute">
+            <parent link="iiwa7_gripper_base_link"/>
+            <child link="iiwa7_gripper_finger2_inner_knuckle_link"/>
             <axis xyz="0 0 1"/>
             <origin xyz="0.06142 -0.0127 0" rpy="0 0 0"/>
             <limit lower="0.0" upper="1.0" velocity="100.0" effort="0.1"/>
-            <mimic joint="${prefix}gripper_finger1_inner_knuckle_joint" offset="0"/>
-        </joint>
-        <link name="${prefix}gripper_finger1_inner_knuckle_link">
+            <mimic joint="iiwa7_gripper_finger1_inner_knuckle_joint" offset="0"/>
+        </joint>
+        <link name="iiwa7_gripper_finger1_inner_knuckle_link">
             <visual>
                 <geometry>
@@ -203,13 +203,13 @@
             </inertial>
         </link>
-        <gazebo reference="${prefix}gripper_finger1_inner_knuckle_link">
-            <implicitSpringDamper>1</implicitSpringDamper>
-            <mu1>100000</mu1>
-            <mu2>100000</mu2>
-            <kp>100000000.0</kp>
-            <kd>1.0</kd>
-            <self_collide>0</self_collide>
-        </gazebo>
-        <link name="${prefix}gripper_finger2_inner_knuckle_link">
+        <gazebo reference="iiwa7_gripper_finger1_inner_knuckle_link">
+            <implicitSpringDamper>1</implicitSpringDamper>
+            <mu1>100000</mu1>
+            <mu2>100000</mu2>
+            <kp>100000000.0</kp>
+            <kd>1.0</kd>
+            <self_collide>0</self_collide>
+        </gazebo>
+        <link name="iiwa7_gripper_finger2_inner_knuckle_link">
             <visual>
                 <geometry>
@@ -230,29 +230,29 @@
             </inertial>
         </link>
-        <gazebo reference="${prefix}gripper_finger2_inner_knuckle_link">
-            <implicitSpringDamper>1</implicitSpringDamper>
-            <mu1>100000</mu1>
-            <mu2>100000</mu2>
-            <kp>100000000.0</kp>
-            <kd>1.0</kd>
-            <self_collide>0</self_collide>
-        </gazebo>
-        <joint name="${prefix}gripper_finger1_finger_tip_joint" type="revolute">
-            <parent link="${prefix}gripper_finger1_inner_knuckle_link"/>
-            <child link="${prefix}gripper_finger1_finger_tip_link"/>
+        <gazebo reference="iiwa7_gripper_finger2_inner_knuckle_link">
+            <implicitSpringDamper>1</implicitSpringDamper>
+            <mu1>100000</mu1>
+            <mu2>100000</mu2>
+            <kp>100000000.0</kp>
+            <kd>1.0</kd>
+            <self_collide>0</self_collide>
+        </gazebo>
+        <joint name="iiwa7_gripper_finger1_finger_tip_joint" type="revolute">
+            <parent link="iiwa7_gripper_finger1_inner_knuckle_link"/>
+            <child link="iiwa7_gripper_finger1_finger_tip_link"/>
             <axis xyz="0 0 1"/>
             <origin xyz="0.04303959807 -0.03759940821 0.0" rpy="0.0 0.0 0.0"/>
             <limit lower="-1.0" upper="0.0" velocity="100.0" effort="0.1"/>
-            <mimic joint="${prefix}gripper_finger1_inner_knuckle_joint" multiplier="-1" offset="0"/>
-        </joint>
-        <joint name="${prefix}gripper_finger2_finger_tip_joint" type="revolute">
-            <parent link="${prefix}gripper_finger2_inner_knuckle_link"/>
-            <child link="${prefix}gripper_finger2_finger_tip_link"/>
+            <mimic joint="iiwa7_gripper_finger1_inner_knuckle_joint" multiplier="-1" offset="0"/>
+        </joint>
+        <joint name="iiwa7_gripper_finger2_finger_tip_joint" type="revolute">
+            <parent link="iiwa7_gripper_finger2_inner_knuckle_link"/>
+            <child link="iiwa7_gripper_finger2_finger_tip_link"/>
             <axis xyz="0 0 1"/>
             <origin rpy="0.0 0.0 0.0" xyz="0.04303959807 -0.03759940821  0.0"/>
             <limit lower="-1.0" upper="0.0" velocity="100.0" effort="0.1"/>
-            <mimic joint="${prefix}gripper_finger1_inner_knuckle_joint" multiplier="-1" offset="0"/>
-        </joint>
-        <link name="${prefix}gripper_finger1_finger_tip_link">
+            <mimic joint="iiwa7_gripper_finger1_inner_knuckle_joint" multiplier="-1" offset="0"/>
+        </joint>
+        <link name="iiwa7_gripper_finger1_finger_tip_link">
             <visual>
                 <geometry>
@@ -273,13 +273,13 @@
             </inertial>
         </link>
-        <gazebo reference="${prefix}gripper_finger1_finger_tip_link">
-            <implicitSpringDamper>1</implicitSpringDamper>
-            <mu1>100000</mu1>
-            <mu2>100000</mu2>
-            <kp>100000000.0</kp>
-            <kd>1.0</kd>
-            <self_collide>0</self_collide>
-        </gazebo>
-        <link name="${prefix}gripper_finger2_finger_tip_link">
+        <gazebo reference="iiwa7_gripper_finger1_finger_tip_link">
+            <implicitSpringDamper>1</implicitSpringDamper>
+            <mu1>100000</mu1>
+            <mu2>100000</mu2>
+            <kp>100000000.0</kp>
+            <kd>1.0</kd>
+            <self_collide>0</self_collide>
+        </gazebo>
+        <link name="iiwa7_gripper_finger2_finger_tip_link">
             <visual>
                 <geometry>
@@ -300,13 +300,13 @@
             </inertial>
         </link>
-        <gazebo reference="${prefix}gripper_finger2_finger_tip_link">
-            <implicitSpringDamper>1</implicitSpringDamper>
-            <mu1>100000</mu1>
-            <mu2>100000</mu2>
-            <kp>100000000.0</kp>
-            <kd>1.0</kd>
-            <self_collide>0</self_collide>
-        </gazebo>
-        <xacro:robotiq_85_gripper_transmission prefix="${prefix}" />
+        <gazebo reference="iiwa7_gripper_finger2_finger_tip_link">
+            <implicitSpringDamper>1</implicitSpringDamper>
+            <mu1>100000</mu1>
+            <mu2>100000</mu2>
+            <kp>100000000.0</kp>
+            <kd>1.0</kd>
+            <self_collide>0</self_collide>
+        </gazebo>
+        <xacro:robotiq_85_gripper_transmission prefix="iiwa7_" />
         <gazebo>
             <plugin name="gazebo_grasp_fix" filename="libgazebo_grasp_fix.so">
