Commit message: Added "getObjDynamics" function to get the mass matrix and nonlinear dynamic vector of the object.

File: examples/pybullet/gym/pybullet_envs/swe_gym/va_kuka_robot/grasp_object.urdf (robot description, URDF)
Before this commit: robot grasp_object, 1 links, 0 joints
Links:
- link object: mass 1 -> 0.1

Commit message: Increased the mass of the object.

File: examples/pybullet/gym/pybullet_envs/swe_gym/va_kuka_robot/grasp_object.urdf (robot description, URDF)
Before this commit: robot grasp_object, 1 links, 0 joints
Links:
- link object: mass 0.1 -> 1
